File: cad/elec/relaisboard/relaisboard.sch (EAGLE design)
At the start: 28 parts, among them IC1 REG1117, T1 MMUN2233

Commit message: increased cleareance here and there
Parts:
- added C14: 2.2u, rcl:C-EUC1206
Connections:
- net +3V3: now also C14.1
- net NEUTRAL: now also C14.2
Changed lines of the file:
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@@
 <part name="+3V3" library="supply1" deviceset="+3V3" device=""/>
 <part name="C45" library="rcl" deviceset="C-EU" device="C1206" value="2.2u"/>
+<part name="C14" library="rcl" deviceset="C-EU" device="C1206" value="2.2u"/>
 </parts>
 <sheets>
@@
 <instance part="+3V3" gate="G$1" x="160.02" y="114.3"/>
 <instance part="C45" gate="G$1" x="127" y="33.02"/>
+<instance part="C14" gate="G$1" x="208.28" y="63.5"/>
 </instances>
 <busses>
@@
 <wire x1="190.5" y1="55.88" x2="172.72" y2="55.88" width="0.1524" layer="91"/>
 <label x="172.72" y="55.88" size="2.1844" layer="95"/>
+<pinref part="C14" gate="G$1" pin="2"/>
+<wire x1="208.28" y1="58.42" x2="208.28" y2="55.88" width="0.1524" layer="91"/>
+<wire x1="208.28" y1="55.88" x2="190.5" y2="55.88" width="0.1524" layer="91"/>
+<junction x="190.5" y="55.88"/>
 </segment>
 </net>
@@
 <pinref part="IC1" gate="G$1" pin="VOUT"/>
 <pinref part="+3V2" gate="G$1" pin="+3V3"/>
-<wire x1="203.2" y1="68.58" x2="210.82" y2="68.58" width="0.1524" layer="91"/>
+<wire x1="203.2" y1="68.58" x2="208.28" y2="68.58" width="0.1524" layer="91"/>
+<wire x1="208.28" y1="68.58" x2="210.82" y2="68.58" width="0.1524" layer="91"/>
 <wire x1="210.82" y1="68.58" x2="210.82" y2="73.66" width="0.1524" layer="91"/>
-</segment>
-<segment>
+<pinref part="C14" gate="G$1" pin="1"/>
+<wire x1="208.28" y1="68.58" x2="208.28" y2="66.04" width="0.1524" layer="91"/>
+<junction x="208.28" y="68.58"/>
+</segment>
+<segment>

Commit message: added new battery powered board and changed lots of other stuff
Parts:
- C1, C2: DIGIKEY (none) -> 1189-1633-1-ND
- C14, C45: DIGIKEY (none) -> 1276-2723-1-ND
- C3: DIGIKEY (none) -> 399-8979-1-ND
- C6: DIGIKEY (none) -> 493-1043-ND
- C7: DIGIKEY (none) -> 1276-1028-1-ND
- D1: REICHELT (none) -> S 1ML SMD
- D4, D6: REICHELT (none) -> ES 1JL SMD
- D5: DIGIKEY (none) -> BYG20J-E3/TRGICT-ND
- DZ7: DIGIKEY (none) -> 568-3810-1-ND
- IC1: DIGIKEY (none) -> AP1117IE33G-13DICT-ND
- L1: REICHELT (none) -> L-PISG 1,0M
- L2: REICHELT (none) -> L-PISR 1,0M
- R1: DIGIKEY (none) -> CF14JT47R0CT-ND
- R2: DIGIKEY (none) -> 1276-3466-1-ND
- R3: DIGIKEY (none) -> RHM18KCDCT-ND
- R4: DIGIKEY (none) -> 311-1.0ERCT-ND
- R5: DIGIKEY (none) -> 311-68KGRCT-ND
- R6: DIGIKEY (none) -> 311-1.00MLRCT-ND
- R7: DIGIKEY (none) -> 311-100JRCT-ND
- T1: DIGIKEY (none) -> MMUN2233LT1GOSCT-ND
- U$1: DIGIKEY (none) -> 568-9556-1-ND
- U$2: DIGIKEY (none) -> 425-2562-5-ND
