File: cad/elec/ucboard/ucboard.sch (EAGLE design)
At the start: 14 parts

Commit message: added two solder bridges to be attach ether the 8 pin transceiver or the 10 pin transceiver (they are almost pin compatible) and exchanged the connectors for dummy 0.05 inch holes. A debug/flash utility can be built more easily
Parts:
- removed SWD: 5PIN, te_1mm_connector:5PIN
- added DBG: (no value), viskos:005CONTACTS
- added R6, R7: 0R/NA, rcl:R-EU_R0201
- UART: value 5PIN -> (none); device te_1mm_connector:5PIN -> viskos:005CONTACTS
Connections:
- new net N$4: R6.2, R7.2, RF_CONN.1
- net +3V3: now also DBG.P$4, R7.1; no longer RF_CONN.1, SWD.P$4
- net GND: now also DBG.P$5, R6.1; no longer SWD.P$5
- net RESET: now also DBG.P$3; no longer SWD.P$3
- net SWCLK: now also DBG.P$1; no longer SWD.P$1
- net SWDIO: now also DBG.P$2; no longer SWD.P$2
Other:
- note added: "there are two types of transceivers: One with 8 pins and one with 10. Short pin1 to ground if your transceiver has 8 pins short to vcc otherwise"

Commit message: added new battery powered board and changed lots of other stuff
Parts:
- C1, C2: DIGIKEY 1276-1041-1-ND -> 1276-1024-1-ND
Connections:
- net GND: now also U$1.P$1, U$1.P$14, U$1.P$22, U$1.P$30, U$1.P$9
Changed lines of the file:
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@@
 <grid distance="0.1" unitdist="inch" unit="inch" style="lines" multiple="1" display="no" altdistance="0.01" altunitdist="inch" altunit="inch"/>
 <layers>
-<layer number="1" name="Top" color="4" fill="1" visible="yes" active="no"/>
+<layer number="1" name="Top" color="4" fill="1" visible="no" active="no"/>
 <layer number="2" name="Route2" color="1" fill="3" visible="no" active="no"/>
 <layer number="3" name="Route3" color="4" fill="3" visible="no" active="no"/>
 <layer number="14" name="Route14" color="1" fill="6" visible="no" active="no"/>
 <layer number="15" name="Route15" color="4" fill="6" visible="no" active="no"/>
-<layer number="16" name="Bottom" color="1" fill="1" visible="yes" active="no"/>
-<layer number="17" name="Pads" color="2" fill="1" visible="yes" active="no"/>
-<layer number="18" name="Vias" color="2" fill="1" visible="yes" active="no"/>
-<layer number="19" name="Unrouted" color="6" fill="1" visible="yes" active="no"/>
-<layer number="20" name="Dimension" color="15" fill="1" visible="yes" active="no"/>
-<layer number="21" name="tPlace" color="7" fill="1" visible="yes" active="no"/>
-<layer number="22" name="bPlace" color="7" fill="1" visible="yes" active="no"/>
-<layer number="23" name="tOrigins" color="15" fill="1" visible="yes" active="no"/>
-<layer number="24" name="bOrigins" color="15" fill="1" visible="yes" active="no"/>
-<layer number="25" name="tNames" color="7" fill="1" visible="yes" active="no"/>
-<layer number="26" name="bNames" color="7" fill="1" visible="yes" active="no"/>
-<layer number="27" name="tValues" color="7" fill="1" visible="yes" active="no"/>
-<layer number="28" name="bValues" color="7" fill="1" visible="yes" active="no"/>
+<layer number="16" name="Bottom" color="1" fill="1" visible="no" active="no"/>
+<layer number="17" name="Pads" color="2" fill="1" visible="no" active="no"/>
+<layer number="18" name="Vias" color="2" fill="1" visible="no" active="no"/>
+<layer number="19" name="Unrouted" color="6" fill="1" visible="no" active="no"/>
+<layer number="20" name="Dimension" color="15" fill="1" visible="no" active="no"/>
+<layer number="21" name="tPlace" color="7" fill="1" visible="no" active="no"/>
+<layer number="22" name="bPlace" color="7" fill="1" visible="no" active="no"/>
+<layer number="23" name="tOrigins" color="15" fill="1" visible="no" active="no"/>
+<layer number="24" name="bOrigins" color="15" fill="1" visible="no" active="no"/>
+<layer number="25" name="tNames" color="7" fill="1" visible="no" active="no"/>
+<layer number="26" name="bNames" color="7" fill="1" visible="no" active="no"/>
+<layer number="27" name="tValues" color="7" fill="1" visible="no" active="no"/>
+<layer number="28" name="bValues" color="7" fill="1" visible="no" active="no"/>
 <layer number="29" name="tStop" color="7" fill="3" visible="no" active="no"/>
 <layer number="30" name="bStop" color="7" fill="6" visible="no" active="no"/>
@@
 <layer number="35" name="tGlue" color="7" fill="4" visible="no" active="no"/>
 <layer number="36" name="bGlue" color="7" fill="5" visible="no" active="no"/>
-<layer number="37" name="tTest" color="7" fill="1" visible="yes" active="no"/>
-<layer number="38" name="bTest" color="7" fill="1" visible="yes" active="no"/>
+<layer number="37" name="tTest" color="7" fill="1" visible="no" active="no"/>
+<layer number="38" name="bTest" color="7" fill="1" visible="no" active="no"/>
 <layer number="39" name="tKeepout" color="4" fill="11" visible="no" active="no"/>
 <layer number="40" name="bKeepout" color="1" fill="11" visible="no" active="no"/>
@@
 <layer number="44" name="Drills" color="7" fill="1" visible="no" active="no"/>
 <layer number="45" name="Holes" color="7" fill="1" visible="no" active="no"/>
-<layer number="46" name="Milling" color="3" fill="1" visible="yes" active="no"/>
-<layer number="47" name="Measures" color="7" fill="1" visible="yes" active="no"/>
-<layer number="48" name="Document" color="7" fill="1" visible="yes" active="no"/>
-<layer number="49" name="Reference" color="7" fill="1" visible="yes" active="no"/>
-<layer number="51" name="tDocu" color="7" fill="1" visible="yes" active="no"/>
-<layer number="52" name="bDocu" color="7" fill="1" visible="yes" active="no"/>
+<layer number="46" name="Milling" color="3" fill="1" visible="no" active="no"/>
+<layer number="47" name="Measures" color="7" fill="1" visible="no" active="no"/>
+<layer number="48" name="Document" color="7" fill="1" visible="no" active="no"/>
+<layer number="49" name="Reference" color="7" fill="1" visible="no" active="no"/>
+<layer number="51" name="tDocu" color="7" fill="1" visible="no" active="no"/>
+<layer number="52" name="bDocu" color="7" fill="1" visible="no" active="no"/>
 <layer number="91" name="Nets" color="2" fill="1" visible="yes" active="yes"/>
 <layer number="92" name="Busses" color="1" fill="1" visible="yes" active="yes"/>
@@
 <part name="+3V8" library="supply1" deviceset="+3V3" device=""/>
 <part name="C1" library="rcl" deviceset="C-EU" device="C0603" value="1u">
-<attribute name="DIGIKEY" value="1276-1041-1-ND"/>
+<attribute name="DIGIKEY" value="1276-1024-1-ND"/>
 </part>
 <part name="C2" library="rcl" deviceset="C-EU" device="C0603" value="1u">
-<attribute name="DIGIKEY" value="1276-1041-1-ND"/>
+<attribute name="DIGIKEY" value="1276-1024-1-ND"/>
 </part>
 <part name="GND6" library="supply1" deviceset="GND" device=""/>
@@
 <part name="DBG" library="viskos" deviceset="005CONTACTS" device=""/>
 <part name="UART" library="viskos" deviceset="005CONTACTS" device=""/>
+<part name="GND12" library="supply1" deviceset="GND" device=""/>
+<part name="GND13" library="supply1" deviceset="GND" device=""/>
+<part name="GND14" library="supply1" deviceset="GND" device=""/>
+<part name="GND15" library="supply1" deviceset="GND" device=""/>
+<part name="GND16" library="supply1" deviceset="GND" device=""/>
 </parts>
 <sheets>
@@
 <instance part="DBG" gate="G$1" x="226.06" y="96.52"/>
 <instance part="UART" gate="G$1" x="228.6" y="68.58"/>
+<instance part="GND12" gate="1" x="86.36" y="10.16"/>
+<instance part="GND13" gate="1" x="144.78" y="53.34" rot="R90"/>
+<instance part="GND14" gate="1" x="78.74" y="93.98" rot="R180"/>
+<instance part="GND15" gate="1" x="73.66" y="10.16"/>
+<instance part="GND16" gate="1" x="45.72" y="66.04" rot="R180"/>
 </instances>
 <busses>
@@
 <wire x1="45.72" y1="157.48" x2="48.26" y2="157.48" width="0.1524" layer="91"/>
 </segment>
+<segment>
+<pinref part="GND14" gate="1" pin="GND"/>
+<pinref part="U$1" gate="G$1" pin="P$30"/>
+<wire x1="78.74" y1="91.44" x2="78.74" y2="68.58" width="0.1524" layer="91"/>
+</segment>
+<segment>
+<pinref part="GND13" gate="1" pin="GND"/>
+<pinref part="U$1" gate="G$1" pin="P$22"/>
+<wire x1="142.24" y1="53.34" x2="114.3" y2="53.34" width="0.1524" layer="91"/>
+</segment>
+<segment>
+<pinref part="GND12" gate="1" pin="GND"/>
+<pinref part="U$1" gate="G$1" pin="P$14"/>
+<wire x1="86.36" y1="12.7" x2="86.36" y2="30.48" width="0.1524" layer="91"/>
+</segment>
+<segment>
+<pinref part="GND15" gate="1" pin="GND"/>
+<pinref part="U$1" gate="G$1" pin="P$9"/>
+<wire x1="73.66" y1="12.7" x2="73.66" y2="30.48" width="0.1524" layer="91"/>
+</segment>
+<segment>
+<pinref part="GND16" gate="1" pin="GND"/>
+<wire x1="45.72" y1="63.5" x2="45.72" y2="58.42" width="0.1524" layer="91"/>
+<pinref part="U$1" gate="G$1" pin="P$1"/>
+<wire x1="45.72" y1="58.42" x2="50.8" y2="58.42" width="0.1524" layer="91"/>
+</segment>
 </net>
