File: cad/elec/stm_ucboard/stm_ucboard.sch (EAGLE design)
At the start: 21 parts

Commit message: chagned attribute
Parts:
- IO_CONN: DIGIKEY 609-3243-ND -> 952-2124-ND
Changed lines of the file:
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@@
 <part name="GND4" library="supply1" deviceset="GND" device=""/>
 <part name="IO_CONN" library="pinhead" deviceset="PINHD-2X5" device="">
-<attribute name="DIGIKEY" value="609-3243-ND"/>
+<attribute name="DIGIKEY" value="952-2124-ND"/>
 </part>
 <part name="+3V6" library="supply1" deviceset="+3V3" device=""/>

Commit message: added pullup/pulldown resistors to the rf pins ; connected PA0 (WKUP1) to external IO interface
Parts:
- added R10, R3, R8, R9: 1M, rcl:R-EU_R0402
- R2: DIGIKEY 311-1.00MLRCT-ND -> 1276-4448-1-ND
Connections:
- net +3V3: now also R3.2
- net GND: now also R10.1, R8.2, R9.1
- net IO_2: now also U$1.PA0
- net RF_CE: now also R9.2
- net RF_CSN: now also R3.1
- net RF_MO: now also R8.1
- net RF_SCK: now also R10.2
Other:
- note added: "This is the WKUP pin"
- moved on the sheet: R6
Changed lines of the file:
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@@
 <part name="GND5" library="supply1" deviceset="GND" device=""/>
 <part name="R2" library="rcl" deviceset="R-EU_" device="R0402" value="1M">
-<attribute name="DIGIKEY" value="311-1.00MLRCT-ND"/>
+<attribute name="DIGIKEY" value="1276-4448-1-ND"/>
 </part>
 <part name="GND7" library="supply1" deviceset="GND" device=""/>
@@
 <part name="C2" library="rcl" deviceset="C-EU" device="C0603" value="100n">
 <attribute name="DIGIKEY" value="399-1095-1-ND"/>
+</part>
+<part name="R3" library="rcl" deviceset="R-EU_" device="R0402" value="1M">
+<attribute name="DIGIKEY" value="1276-4448-1-ND"/>
+</part>
+<part name="+3V1" library="supply1" deviceset="+3V3" device=""/>
+<part name="R8" library="rcl" deviceset="R-EU_" device="R0402" value="1M">
+<attribute name="DIGIKEY" value="1276-4448-1-ND"/>
+</part>
+<part name="GND2" library="supply1" deviceset="GND" device=""/>
+<part name="R9" library="rcl" deviceset="R-EU_" device="R0402" value="1M">
+<attribute name="DIGIKEY" value="1276-4448-1-ND"/>
+</part>
+<part name="R10" library="rcl" deviceset="R-EU_" device="R0402" value="1M">
+<attribute name="DIGIKEY" value="1276-4448-1-ND"/>
 </part>
 </parts>
@@
 your transceiver has 8
 pins short to vcc otherwise</text>
+<text x="22.86" y="-66.04" size="1.778" layer="97">This is the WKUP pin</text>
 </plain>
 <instances>
@@
 <attribute name="DIGIKEY" x="215.9" y="132.08" size="1.778" layer="96" display="off"/>
 </instance>
-<instance part="GND11" gate="1" x="45.72" y="152.4"/>
-<instance part="R6" gate="G$1" x="53.34" y="157.48"/>
+<instance part="GND11" gate="1" x="38.1" y="144.78"/>
+<instance part="R6" gate="G$1" x="48.26" y="157.48"/>
 <instance part="R7" gate="G$1" x="53.34" y="160.02"/>
 <instance part="DBG" gate="G$1" x="226.06" y="96.52">
@@
 <instance part="C2" gate="G$1" x="33.02" y="-43.18" rot="R180">
 <attribute name="DIGIKEY" x="33.02" y="-43.18" size="1.778" layer="96" rot="R180" display="off"/>
+</instance>
+<instance part="R3" gate="G$1" x="119.38" y="154.94">
+<attribute name="DIGIKEY" x="119.38" y="154.94" size="1.778" layer="96" display="off"/>
+</instance>
+<instance part="+3V1" gate="G$1" x="129.54" y="154.94" rot="R270"/>
+<instance part="R8" gate="G$1" x="119.38" y="152.4">
+<attribute name="DIGIKEY" x="119.38" y="152.4" size="1.778" layer="96" display="off"/>
+</instance>
+<instance part="GND2" gate="1" x="127" y="147.32"/>
+<instance part="R9" gate="G$1" x="48.26" y="154.94">
+<attribute name="DIGIKEY" x="48.26" y="154.94" size="1.778" layer="96" display="off"/>
+</instance>
+<instance part="R10" gate="G$1" x="48.26" y="152.4">
+<attribute name="DIGIKEY" x="48.26" y="152.4" size="1.778" layer="96" display="off"/>
 </instance>
 </instances>
@@
 <segment>
 <pinref part="GND11" gate="1" pin="GND"/>
-<wire x1="45.72" y1="154.94" x2="45.72" y2="157.48" width="0.1524" layer="91"/>
+<wire x1="38.1" y1="147.32" x2="38.1" y2="152.4" width="0.1524" layer="91"/>
 <pinref part="R6" gate="G$1" pin="1"/>
-<wire x1="45.72" y1="157.48" x2="48.26" y2="157.48" width="0.1524" layer="91"/>
+<wire x1="38.1" y1="152.4" x2="38.1" y2="154.94" width="0.1524" layer="91"/>
+<wire x1="38.1" y1="154.94" x2="38.1" y2="157.48" width="0.1524" layer="91"/>
+<wire x1="38.1" y1="157.48" x2="43.18" y2="157.48" width="0.1524" layer="91"/>
+<pinref part="R9" gate="G$1" pin="1"/>
+<wire x1="43.18" y1="154.94" x2="38.1" y2="154.94" width="0.1524" layer="91"/>
+<junction x="38.1" y="154.94"/>
+<pinref part="R10" gate="G$1" pin="1"/>
+<wire x1="43.18" y1="152.4" x2="38.1" y2="152.4" width="0.1524" layer="91"/>
+<junction x="38.1" y="152.4"/>
 </segment>
 <segment>
@@
 <wire x1="-30.48" y1="-17.78" x2="-22.86" y2="-17.78" width="0.1524" layer="91"/>
 <junction x="-22.86" y="-17.78"/>
+</segment>
+<segment>
+<pinref part="R8" gate="G$1" pin="2"/>
+<pinref part="GND2" gate="1" pin="GND"/>
+<wire x1="124.46" y1="152.4" x2="127" y2="152.4" width="0.1524" layer="91"/>
+<wire x1="127" y1="152.4" x2="127" y2="149.86" width="0.1524" layer="91"/>
 </segment>
 </net>
@@
 <junction x="101.6" y="-55.88"/>
 </segment>
+<segment>
+<pinref part="R3" gate="G$1" pin="2"/>
+<pinref part="+3V1" gate="G$1" pin="+3V3"/>
+<wire x1="124.46" y1="154.94" x2="127" y2="154.94" width="0.1524" layer="91"/>
+</segment>
 </net>
 <net name="RESET" class="0">
@@
 <net name="RF_CE" class="0">
 <segment>
-<wire x1="76.2" y1="154.94" x2="55.88" y2="154.94" width="0.1524" layer="91"/>
+<wire x1="76.2" y1="154.94" x2="53.34" y2="154.94" width="0.1524" layer="91"/>
 <label x="55.88" y="154.94" size="1.778" layer="95"/>
 <pinref part="RF_CONN" gate="A" pin="3"/>
+<pinref part="R9" gate="G$1" pin="2"/>
 </segment>
 <segment>
@@
 <net name="RF_SCK" class="0">
 <segment>
-<wire x1="76.2" y1="152.4" x2="55.88" y2="152.4" width="0.1524" layer="91"/>
+<wire x1="76.2" y1="152.4" x2="53.34" y2="152.4" width="0.1524" layer="91"/>
 <label x="55.88" y="152.4" size="1.778" layer="95"/>
 <pinref part="RF_CONN" gate="A" pin="5"/>
+<pinref part="R10" gate="G$1" pin="2"/>
 </segment>
 <segment>
@@
 <net name="RF_CSN" class="0">
 <segment>
-<wire x1="83.82" y1="154.94" x2="106.68" y2="154.94" width="0.1524" layer="91"/>
+<wire x1="83.82" y1="154.94" x2="114.3" y2="154.94" width="0.1524" layer="91"/>
 <label x="96.52" y="154.94" size="1.778" layer="95"/>
 <pinref part="RF_CONN" gate="A" pin="4"/>
+<pinref part="R3" gate="G$1" pin="1"/>
 </segment>
 <segment>
@@
 <net name="RF_MO" class="0">
 <segment>
-<wire x1="83.82" y1="152.4" x2="106.68" y2="152.4" width="0.1524" layer="91"/>
+<wire x1="83.82" y1="152.4" x2="114.3" y2="152.4" width="0.1524" layer="91"/>
 <label x="96.52" y="152.4" size="1.778" layer="95"/>
 <pinref part="RF_CONN" gate="A" pin="6"/>
+<pinref part="R8" gate="G$1" pin="1"/>
 </segment>
 <segment>
@@
 <label x="137.16" y="-35.56" size="1.778" layer="95"/>
 </segment>
+<segment>
+<pinref part="U$1" gate="G$1" pin="PA0"/>
+<wire x1="48.26" y1="-35.56" x2="45.72" y2="-35.56" width="0.1524" layer="91"/>
+<wire x1="45.72" y1="-35.56" x2="45.72" y2="-63.5" width="0.1524" layer="91"/>
+<wire x1="45.72" y1="-63.5" x2="27.94" y2="-63.5" width="0.1524" layer="91"/>
+<label x="27.94" y="-63.5" size="1.778" layer="95"/>
+</segment>
 </net>
 <net name="LED_R" class="0">
@@
 <wire x1="60.96" y1="160.02" x2="60.96" y2="157.48" width="0.1524" layer="91"/>
 <pinref part="R6" gate="G$1" pin="2"/>
-<wire x1="60.96" y1="157.48" x2="58.42" y2="157.48" width="0.1524" layer="91"/>
+<wire x1="60.96" y1="157.48" x2="53.34" y2="157.48" width="0.1524" layer="91"/>
 <pinref part="RF_CONN" gate="A" pin="1"/>
 <wire x1="60.96" y1="157.48" x2="76.2" y2="157.48" width="0.1524" layer="91"/>
