File: cad/elec/battery_powered_devel_board/battery_powered_devel_board.sch (EAGLE design)
At the start: 16 parts

Commit message: changed battery sensing line on battery board to fit stm uc board
Connections:
- net IO_4: no longer R1.2
- net IO_6: now also R1.2
Changed lines of the file:
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@@
 <pinref part="PAD5" gate="P" pin="P"/>
-</segment>
-<segment>
-<pinref part="R1" gate="G$1" pin="2"/>
-<wire x1="55.88" y1="129.54" x2="55.88" y2="132.08" width="0.1524" layer="91"/>
-<wire x1="55.88" y1="132.08" x2="73.66" y2="132.08" width="0.1524" layer="91"/>
-<label x="68.58" y="132.08" size="1.778" layer="95"/>
 </segment>
 </net>
@@
 <pinref part="PAD7" gate="P" pin="P"/>
 </segment>
+<segment>
+<pinref part="R1" gate="G$1" pin="2"/>
+<wire x1="55.88" y1="129.54" x2="55.88" y2="132.08" width="0.1524" layer="91"/>
+<wire x1="55.88" y1="132.08" x2="81.28" y2="132.08" width="0.1524" layer="91"/>
+<label x="76.2" y="132.08" size="1.778" layer="95"/>
+</segment>
 </net>

Commit message: corrected the attributes
Parts:
- JP1: DIGIKEY (none) -> S6105-ND
Changed lines of the file:
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@@
 </classes>
 <parts>
-<part name="JP1" library="pinhead" deviceset="PINHD-2X5" device=""/>
+<part name="JP1" library="pinhead" deviceset="PINHD-2X5" device="">
+<attribute name="DIGIKEY" value="S6105-ND"/>
+</part>
 <part name="+3V1" library="supply1" deviceset="+3V3" device=""/>
 <part name="GND1" library="supply1" deviceset="GND" device=""/>
@@
 </plain>
 <instances>
-<instance part="JP1" gate="A" x="60.96" y="78.74"/>
+<instance part="JP1" gate="A" x="60.96" y="78.74">
+<attribute name="DIGIKEY" x="60.96" y="78.74" size="1.778" layer="96" display="off"/>
+</instance>
 <instance part="+3V1" gate="G$1" x="43.18" y="73.66" rot="R90"/>
 <instance part="GND1" gate="1" x="78.74" y="66.04"/>
